File: Hardware/USG.kicad_pcb (KiCad board)
At the start: 2 copper layers, 78 x 29.6 mm, 70 parts, among them P1 USB_A_PLUG, P2 USB_A_SOCKET, P3 USB_OTG, U1 NUP4114, U2 STM32F401xB, U3 AZ1117CH-3.3, U4 STM32F401xB, U5 NUP4114, Y1 8MHz, Y2 8MHz

Commit message: Hardware v1.0 beta complete, ready for fabrication
Parts:
- added ?: Symbol_OSHW-Logo_SilkScreen, Symbols:Symbol_OSHW-Logo_SilkScreen, B.Cu at (130.7, 107.1)
- P3: footprint USG_footprints:USB_Micro-B-SMD -> Connect:USB_Micro-B; moved to F.Cu
- moved ID_DNST1 58.2 mm to (161.9, 106.6), turned to 90 degrees
- moved C28 55.1 mm to (177.4, 100.6), turned to 180 degrees
- moved ID_BOARD2 53.3 mm to (163.6, 106.6), turned to 90 degrees
- moved C18 53.3 mm to (159.0, 101.9), turned to 180 degrees
- moved C16 50.3 mm to (154.4, 103.8), turned to 180 degrees
- moved ID_BOARD1 48.6 mm to (165.1, 106.6), turned to 90 degrees
- moved R14 46.8 mm to (171.7, 119.0), turned to 180 degrees
- moved R9 46.5 mm to (172.2, 112.1), turned to 270 degrees
- moved C25 46.5 mm to (156.7, 106.6), turned to 270 degrees
- moved P2 46.4 mm to (180.2, 111.0)
- moved C27 45.7 mm to (180.0, 117.7), turned to 90 degrees
- moved C20 45.6 mm to (157.4, 116.3)
- moved R15 45.3 mm to (171.7, 117.2), turned to 180 degrees
- moved JTAG_DNST 44.3 mm to (176.8, 115.2), turned to 180 degrees
- moved Y2 44.0 mm to (164.6, 98.2), turned to 180 degrees
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- renumbered BOOT_DNST1 to BOOT_DNST, BOOT_UPST1 to BOOT_UPST, FAULT_DNST1 to FAULT_DNST, FAULT_UPST1 to FAULT_UPST, ID_DNST_BOARD0 to ID_BOARD0, ID_UPST_BOARD0 to ID_BOARD0, ID_DNST_BOARD1 to ID_BOARD1, ID_UPST_BOARD1 to ID_BOARD1, ID_DNST_BOARD2 to ID_BOARD2, ID_UPST_BOARD2 to ID_BOARD2, JTAG_DNST1 to JTAG_DNST, JTAG_UPST1 to JTAG_UPST, RESET1 to RESET
Routing:
- net GND: track 206.4 -> 490.8 mm, vias 21 -> 69
- net +3V3: track 113.8 -> 210.0 mm, vias 6 -> 4
- net /RESET_DNST: track 14.9 -> 61.7 mm
- net +5V: track 72.5 -> 115.9 mm, vias 6 -> 10
- net Net-(P2-Pad2): track 0.00 -> 27.3 mm
- net Net-(P2-Pad3): track 0.00 -> 26.8 mm
- net /SPI_MOSI: track 19.6 -> 37.4 mm, vias 1 -> 2
- net /SPI_TX_OK: track 20.0 -> 37.3 mm, vias 1 -> 2
- net /SPI_MISO: track 19.6 -> 36.6 mm, vias 1 -> 2
- net /SPI_NSS: track 19.6 -> 36.6 mm, vias 1 -> 2
- net /SPI_SCK: track 19.7 -> 36.6 mm, vias 1 -> 2
- net (no net): track 0.00 -> 11.4 mm
- net Net-(C17-Pad1): track 0.00 -> 10.8 mm
- net Net-(R14-Pad2): track 0.00 -> 10.6 mm
- net Net-(BOOT_DNST1-Pad1): track 0.00 -> 10.3 mm
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- added copper zone on B.Cu, net GND
- added copper zone on F.Cu, net GND
Other:
- board size 78 x 29.6 mm -> 71 x 25 mm
- rule pad_to_mask_clearance: 0.2 -> 0.1
- board text added: "Designed & assembled in New Zealand"
- board text added: "Downstream"
- board text added: "USG v1.0 beta"
- board text added: "Upstream"
- board text added: "github.com/robertfisk/usg"
